Commit message: Change Gazzebo wheel_base_distance 0.174

File: src/puzzlebot_description/urdf/mcr2_robots/hacker_ed/parameters_hacker_ed.xacro (robot description, xacro)
@@ -5,5 +5,5 @@
     <!--Puzzlebot parameters-->
         <!--General parameters-->
-            <xacro:property name="wheel_base_distance" value="0.19"/>
+            <xacro:property name="wheel_base_distance" value="0.174"/>
     <!--Chassis-->
         <!--Chassis Inertial/Collision parameters-->

File: src/puzzlebot_description/urdf/mcr2_robots/jetson_ed/parameters_jetson_ed.xacro (robot description, xacro)
@@ -5,5 +5,5 @@
     <!--Puzzlebot parameters-->
         <!--General parameters-->
-            <xacro:property name="wheel_base_distance" value="0.19"/>
+            <xacro:property name="wheel_base_distance" value="0.174"/>
     <!--Chassis-->
         <!--Chassis Inertial/Collision parameters-->

File: src/puzzlebot_description/urdf/mcr2_robots/jetson_lidar_ed/parameters_jetson_lidar_ed.xacro (robot description, xacro)
@@ -5,5 +5,5 @@
     <!--Puzzlebot parameters-->
         <!--General parameters-->
-            <xacro:property name="wheel_base_distance" value="0.19"/>
+            <xacro:property name="wheel_base_distance" value="0.174"/>
     <!--Chassis-->
         <!--Chassis Inertial/Collision parameters-->
